File: KiCAD/usbc-data-splitter.kicad_sch (KiCad schematic)
At the start: 0 parts

Commit message: Fix journal and add a gitignore.
Parts:
- added J1: Data, Connector_USB:USB_C_Receptacle_Amphenol_12401610E4-2A, symbol Connector:USB_C_Receptacle
- added J2: Power, Connector_USB:USB_C_Receptacle_Amphenol_12401610E4-2A, symbol Connector:USB_C_Receptacle_USB2.0_16P
- added P1: Combined, Connector_USB:USB_C_Receptacle_Amphenol_12401610E4-2A, symbol Connector:USB_C_Plug
Connections:
- new net: J1.A4 (VBUS), J1.A9 (VBUS), J1.B4 (VBUS), J1.B9 (VBUS)
- new net CC: J2.A5 (CC1), P1.A5 (CC)
- new net D_N: J1.A7 (D-), J1.B7 (D-), P1.A7 (D-)
- new net D_P: J1.A6 (D+), J1.B6 (D+), P1.A6 (D+)
- new net GND: J1.A1 (GND), J1.A12 (GND), J1.B1 (GND), J1.B12 (GND), J1.S1 (SHIELD), J2.A1 (GND), J2.A12 (GND), J2.B1 (GND), J2.B12 (GND), J2.S1 (SHIELD), P1.A1 (GND), P1.A12 (GND), P1.B1 (GND), P1.B12 (GND), P1.S1 (SHIELD)
- new net RX1_N: J1.B10 (RX1-), P1.B10 (RX1-)
- new net RX1_P: J1.B11 (RX1+), P1.B11 (RX1+)
- new net RX2_N: J1.A10 (RX2-), P1.A10 (RX2-)
- new net RX2_P: J1.A11 (RX2+), P1.A11 (RX2+)
- new net SBU1: J2.A8 (SBU1), P1.A8 (SBU1)
- new net SBU2: J2.B8 (SBU2), P1.B8 (SBU2)
- new net TX1_N: J1.A3 (TX1-), P1.A3 (TX1-)
- new net TX1_P: J1.A2 (TX1+), P1.A2 (TX1+)
- new net TX2_N: J1.B3 (TX2-), P1.B3 (TX2-)
- new net TX2_P: J1.B2 (TX2+), P1.B2 (TX2+)
- new net VBUS: J2.A4 (VBUS), J2.A9 (VBUS), J2.B4 (VBUS), J2.B9 (VBUS), P1.A4 (VBUS), P1.A9 (VBUS), P1.B4 (VBUS), P1.B9 (VBUS)
- new net VCON: J2.B5 (CC2), P1.B5 (VCONN)
- no-connect marks 0 -> 9
Other:
- note added: "Combined"
- note added: "Separate"
